File: otavca.sch (KiCad schematic (older format))
At the start: 5 parts

Commit message: start vca section
Parts:
- added C?: C, symbol Device:C
- added J?: AudioJack2_Dual_Ground_Switch, symbol Connector:AudioJack2_Dual_Ground_Switch
- added R? (x2): 12k, symbol Device:R
- added R?: 27k, symbol Device:R
- added RV?: 1k, symbol Device:R_POT
- added RV?: 1M, symbol Device:R_POT
- added U?: LM13700, symbol Amplifier_Operational:LM13700
- added U? (x2): TL074, symbol Amplifier_Operational:TL074
Connections:
- net +12V: now also R?.2
- net GND: now also J?.G, RV?.2
- new net: C?.2, RV?.1, U?.12, U?.6 (-)
- new net: RV?.1, U?.13 (-)
- new net: R?.1, RV?.3, U?.14 (+)
- new net: R?.1, U?.15 (DIODE_BIAS)
- new net: C?.1, R?.1, U?.7
- new net: J?.T1, R?.2
- new net: R?.2, RV?.2, RV?.3
- no-connect marks 0 -> 3
Changed lines of the file:
@@
 Wire Wire Line
 	3025 7125 2875 7125
+$Comp
+L Amplifier_Operational:LM13700 U?
+U 1 1 61686809
+P 3750 2675
+F 0 "U?" H 3750 3042 50  0000 C CNN
+F 1 "LM13700" H 3750 2951 50  0000 C CNN
+F 2 "" H 3450 2700 50  0001 C CNN
+F 3 "http://www.ti.com/lit/ds/symlink/lm13700.pdf" H 3450 2700 50  0001 C CNN
+	1    3750 2675
+	1    0    0    -1
+$EndComp
+$Comp
+L Amplifier_Operational:TL074 U?
+U 1 1 6168765B
+P 3325 3750
+F 0 "U?" H 3325 4117 50  0000 C CNN
+F 1 "TL074" H 3325 4026 50  0000 C CNN
+F 2 "" H 3275 3850 50  0001 C CNN
+F 3 "http://www.ti.com/lit/ds/symlink/tl071.pdf" H 3375 3950 50  0001 C CNN
+	1    3325 3750
+	1    0    0    -1
+$EndComp
+$Comp
+L Amplifier_Operational:TL074 U?
+U 2 1 616886AF
+P 5025 2825
+F 0 "U?" H 5025 2458 50  0000 C CNN
+F 1 "TL074" H 5025 2549 50  0000 C CNN
+F 2 "" H 4975 2925 50  0001 C CNN
+F 3 "http://www.ti.com/lit/ds/symlink/tl071.pdf" H 5075 3025 50  0001 C CNN
+	2    5025 2825
+	1    0    0    1
+$EndComp
+$Comp
+L Device:R R?
+U 1 1 6168BEA1
+P 3300 2675
+F 0 "R?" V 3093 2675 50  0000 C CNN
+F 1 "12k" V 3184 2675 50  0000 C CNN
+F 2 "" V 3230 2675 50  0001 C CNN
+F 3 "~" H 3300 2675 50  0001 C CNN
+	1    3300 2675
+	0    1    1    0
+$EndComp
+$Comp
+L Device:R R?
+U 1 1 6168C7D2
+P 2825 2775
+F 0 "R?" V 2618 2775 50  0000 C CNN
+F 1 "27k" V 2709 2775 50  0000 C CNN
+F 2 "" V 2755 2775 50  0001 C CNN
+F 3 "~" H 2825 2775 50  0001 C CNN
+	1    2825 2775
+	0    1    1    0
+$EndComp
+Wire Wire Line
+	3450 2775 3025 2775
+$Comp
+L power:+12V #PWR?
+U 1 1 6168D5F3
+P 3150 2675
+F 0 "#PWR?" H 3150 2525 50  0001 C CNN
+F 1 "+12V" H 3165 2848 50  0000 C CNN
+F 2 "" H 3150 2675 50  0001 C CNN
+F 3 "" H 3150 2675 50  0001 C CNN
+	1    3150 2675
+	1    0    0    -1
+$EndComp
+$Comp
+L Device:R_POT RV?
+U 1 1 6168E012
+P 3025 2350
+F 0 "RV?" H 2955 2396 50  0000 R CNN
+F 1 "1k" H 2955 2305 50  0000 R CNN
+F 2 "" H 3025 2350 50  0001 C CNN
+F 3 "~" H 3025 2350 50  0001 C CNN
+	1    3025 2350
+	1    0    0    -1
+$EndComp
+$Comp
+L power:GND #PWR?
+U 1 1 6168EA52
+P 3175 2350
+F 0 "#PWR?" H 3175 2100 50  0001 C CNN
+F 1 "GND" V 3180 2222 50  0000 R CNN
+F 2 "" H 3175 2350 50  0001 C CNN
+F 3 "" H 3175 2350 50  0001 C CNN
+	1    3175 2350
+	0    -1   -1   0
+$EndComp
+Wire Wire Line
+	3450 2575 3450 2200
+Wire Wire Line
+	3450 2200 3025 2200
+Wire Wire Line
+	3025 2500 3025 2775
+Connection ~ 3025 2775
+Wire Wire Line
+	3025 2775 2975 2775
+$Comp
+L Connector:AudioJack2_Dual_Ground_Switch J?
+U 1 1 61690241
+P 1825 2650
+F 0 "J?" H 1832 3075 50  0000 C CNN
+F 1 "AudioJack2_Dual_Ground_Switch" H 1832 2984 50  0000 C CNN
+F 2 "" H 1775 2850 50  0001 C CNN
+F 3 "~" H 1775 2850 50  0001 C CNN
+	1    1825 2650
+	1    0    0    -1
+$EndComp
+NoConn ~ 2025 2550
+NoConn ~ 2025 2450
+NoConn ~ 2025 2750
+$Comp
+L power:GND #PWR?
+U 1 1 61692CF8
+P 1825 2950
+F 0 "#PWR?" H 1825 2700 50  0001 C CNN
+F 1 "GND" H 1830 2777 50  0000 C CNN
+F 2 "" H 1825 2950 50  0001 C CNN
+F 3 "" H 1825 2950 50  0001 C CNN
+	1    1825 2950
+	1    0    0    -1
+$EndComp
+Wire Wire Line
+	2675 2775 2150 2775
+Wire Wire Line
+	2150 2775 2150 2650
+Wire Wire Line
+	2150 2650 2025 2650
+Wire Wire Line
+	4050 2675 4525 2675
+Wire Wire Line
+	4725 2675 4725 2725
+$Comp
+L Device:C C?
+U 1 1 61694D8B
+P 5000 1825
+F 0 "C?" V 4748 1825 50  0000 C CNN
+F 1 "C" V 4839 1825 50  0000 C CNN
+F 2 "" H 5038 1675 50  0001 C CNN
+F 3 "~" H 5000 1825 50  0001 C CNN
+	1    5000 1825
+	0    1    1    0
+$EndComp
+Wire Wire Line
+	4525 2675 4525 2225
+Wire Wire Line
+	4525 1825 4850 1825
+Connection ~ 4525 2675
+Wire Wire Line
+	4525 2675 4725 2675
+Wire Wire Line
+	5150 1825 5475 1825
+Wire Wire Line
+	5475 1825 5475 2225
+Wire Wire Line
+	5475 2825 5325 2825
+$Comp
+L Device:R_POT RV?
+U 1 1 61696310
+P 4750 2225
+F 0 "RV?" V 4635 2225 50  0000 C CNN
+F 1 "1M" V 4544 2225 50  0000 C CNN
+F 2 "" H 4750 2225 50  0001 C CNN
+F 3 "~" H 4750 2225 50  0001 C CNN
+	1    4750 2225
+	0    -1   -1   0
+$EndComp
+$Comp
+L Device:R R?
+U 1 1 616968C7
+P 5175 2225
+F 0 "R?" V 4968 2225 50  0000 C CNN
+F 1 "12k" V 5059 2225 50  0000 C CNN
+F 2 "" V 5105 2225 50  0001 C CNN
+F 3 "~" H 5175 2225 50  0001 C CNN
+	1    5175 2225
+	0    1    1    0
+$EndComp
+Wire Wire Line
+	5325 2225 5475 2225
+Connection ~ 5475 2225
+Wire Wire Line
+	5475 2225 5475 2825
+Wire Wire Line
+	5025 2225 4900 2225
+Wire Wire Line
+	4600 2225 4525 2225
+Connection ~ 4525 2225
+Wire Wire Line
+	4525 2225 4525 1825
+Wire Wire Line
+	4750 2075 4900 2075
+Wire Wire Line
+	4900 2075 4900 2225
+Connection ~ 4900 2225
 $EndSCHEMATC
